File: _pcb/main_pcb/main_pcb/main_pcb.kicad_pcb (KiCad board)
At the start: 2 copper layers, 185 x 110 mm, 53 parts, among them J1 Conn_01x01_Pin, J2 Conn_01x01_Pin, SW1 SW_Push, SW2 SW_Push, SW3 SW_Push, SW4 SW_Push, SW5 SW_Push, SW6 SW_Push, SW7 SW_Push, SW8 SW_Push, U1 Pico, U2 74HC4051, U3 PCF8575DBR

Commit message: removed all pcb plans
Parts:
- removed C1, C2, C3, C4, C5, C6, C7, C8: C, Capacitor_SMD:C_1206_3216Metric
- removed D1, D2, D3, D4, D5, D6, D7, D8: WS2812B, LED_SMD:LED_WS2812B_PLCC4_5.0x5.0mm_P3.2mm
- removed J1, J2: Conn_01x01_Pin, TestPoint:TestPoint_Pad_3.0x3.0mm
- removed R1, R2, R3, R4: 10k, Potentiometer:Linear_Potentiometer
- removed R10, R11, R12, R13, R14, R15, R16, R17, R18, R19, R20, R5, R6, R7, R8, R9: R, Resistor_SMD:R_1206_3216Metric
- removed SW1, SW2, SW3, SW4, SW5, SW6, SW7, SW8: SW_Push, Button_Switch_Keyboard:SW_Cherry_MX_1.00u_Plate
- removed U1: Pico, MCU_RaspberryPi_and_Boards:RPi_Pico_SMD_TH
- removed U2: 74HC4051, Package_DIP:SMDIP-16_W9.53mm
- removed U3: PCF8575DBR, Package_SO:SSOP-24_5.3x8.2mm_P0.65mm
- removed rotSW1, rotSW2, rotSW3, rotSW4: RotaryEncoder_Switch, Rotary_Encoder:RotaryEncoder_Alps_EC11E-Switch_Vertical_H20mm
Routing:
- net ADC_MUL_PLEX_GPIO_0: track 16.8 -> 0.00 mm
- net ADC_MUL_PLEX_GPIO_1: track 12.4 -> 0.00 mm
- net ADC_MUL_PLEX_GPIO_2: track 7.89 -> 0.00 mm
- removed copper zone on B.Cu, net GND
- removed copper zone on F.Cu, net GND
Other:
- board outline removed

Commit message: bauteile sortiert
Parts:
- added C1: C, Capacitor_SMD:C_1206_3216Metric, F.Cu at (72.2, 116.6)
- added C10: C, Capacitor_SMD:C_1206_3216Metric, F.Cu at (72.2, 133.4)
- added C2: C, Capacitor_SMD:C_1206_3216Metric, F.Cu at (72.2, 120.0)
- added C3: C, Capacitor_SMD:C_1206_3216Metric, F.Cu at (72.2, 123.3)
- added C4: C, Capacitor_SMD:C_1206_3216Metric, F.Cu at (72.2, 126.7)
- added C9: C, Capacitor_SMD:C_1206_3216Metric, F.Cu at (72.2, 130.0)
- added D1: WS2812B, LED_SMD:LED_WS2812B_PLCC4_5.0x5.0mm_P3.2mm, F.Cu at (12.7, 227.5)
- added D10: LED, LED_THT:LED_Rectangular_W3.9mm_H1.9mm, F.Cu at (-96.2, 267.5)
- added D11: LED, LED_THT:LED_Rectangular_W3.9mm_H1.9mm, F.Cu at (-96.2, 271.2)
- added D12: LED, LED_THT:LED_Rectangular_W3.9mm_H1.9mm, F.Cu at (-96.2, 274.8)
- added D13: LED, LED_THT:LED_Rectangular_W3.9mm_H1.9mm, F.Cu at (-96.2, 278.5)
- added D14: LED, LED_THT:LED_Rectangular_W3.9mm_H1.9mm, F.Cu at (-96.2, 282.1)
- added D15: LED, LED_THT:LED_Rectangular_W3.9mm_H1.9mm, F.Cu at (-96.2, 285.8)
- added D16: LED, LED_THT:LED_Rectangular_W3.9mm_H1.9mm, F.Cu at (-96.2, 289.4)
- added D2: WS2812B, LED_SMD:LED_WS2812B_PLCC4_5.0x5.0mm_P3.2mm, F.Cu at (12.7, 234.1)
- added D3: WS2812B, LED_SMD:LED_WS2812B_PLCC4_5.0x5.0mm_P3.2mm, F.Cu at (12.7, 240.8)
- added D4: WS2812B, LED_SMD:LED_WS2812B_PLCC4_5.0x5.0mm_P3.2mm, F.Cu at (12.7, 247.4)
- added D5: WS2812B, LED_SMD:LED_WS2812B_PLCC4_5.0x5.0mm_P3.2mm, F.Cu at (12.7, 254.0)
- added D6: WS2812B, LED_SMD:LED_WS2812B_PLCC4_5.0x5.0mm_P3.2mm, F.Cu at (21.1, 227.5)
- added D7: WS2812B, LED_SMD:LED_WS2812B_PLCC4_5.0x5.0mm_P3.2mm, F.Cu at (21.1, 234.1)
- added D8: WS2812B, LED_SMD:LED_WS2812B_PLCC4_5.0x5.0mm_P3.2mm, F.Cu at (21.1, 240.8)
- added D9: LED, LED_THT:LED_Rectangular_W3.9mm_H1.9mm, F.Cu at (-96.2, 263.9)
- added J1: Conn_01x01_Pin, TestPoint:TestPoint_Pad_3.0x3.0mm, F.Cu at (-217.6, 233.9)
- added J2: Conn_01x01_Pin, TestPoint:TestPoint_Pad_3.0x3.0mm, F.Cu at (-217.6, 238.9)
- added R1: 10k, Potentiometer:Linear_Potentiometer, F.Cu at (-106.2, 123.2)
- added R10: R, Resistor_SMD:R_1206_3216Metric, F.Cu at (72.2, 153.2)
- added R2: 10k, Potentiometer:Linear_Potentiometer, F.Cu at (-94.6, 123.2)
- added R21: 10k, Potentiometer:Linear_Potentiometer, F.Cu at (-59.8, 123.2)
- added R22: R, Inductor_SMD:L_1206_3216Metric_Pad1.22x1.90mm_HandSolder, F.Cu at (-88.9, 263.8)
- added R23: R, Inductor_SMD:L_1206_3216Metric_Pad1.22x1.90mm_HandSolder, F.Cu at (-88.9, 267.2)
- added R24: R, Inductor_SMD:L_1206_3216Metric_Pad1.22x1.90mm_HandSolder, F.Cu at (-88.9, 270.7)
- added R25: R, Inductor_SMD:L_1206_3216Metric_Pad1.22x1.90mm_HandSolder, F.Cu at (-88.9, 274.1)
- added R26: R, Inductor_SMD:L_1206_3216Metric_Pad1.22x1.90mm_HandSolder, F.Cu at (-88.9, 277.6)
- added R27: R, Inductor_SMD:L_1206_3216Metric_Pad1.22x1.90mm_HandSolder, F.Cu at (-88.9, 281.0)
- added R28: R, Inductor_SMD:L_1206_3216Metric_Pad1.22x1.90mm_HandSolder, F.Cu at (-88.9, 284.5)
- added R29: R, Inductor_SMD:L_1206_3216Metric_Pad1.22x1.90mm_HandSolder, F.Cu at (-88.9, 287.9)
- added R3: 10k, Potentiometer:Linear_Potentiometer, F.Cu at (-83.0, 123.2)
- added R4: 10k, Potentiometer:Linear_Potentiometer, F.Cu at (-71.4, 123.2)
- added R5: R, Resistor_SMD:R_1206_3216Metric, F.Cu at (72.2, 136.7)
- added R6: R, Resistor_SMD:R_1206_3216Metric, F.Cu at (72.2, 140.0)
- added R7: R, Resistor_SMD:R_1206_3216Metric, F.Cu at (72.2, 143.3)
- added R8: R, Resistor_SMD:R_1206_3216Metric, F.Cu at (72.2, 146.6)
- added R9: R, Resistor_SMD:R_1206_3216Metric, F.Cu at (72.2, 149.9)
- added SW1: SW_Push, Button_Switch_Keyboard:SW_Cherry_MX_1.00u_Plate, F.Cu at (-157.0, 287.2)
- added SW2: SW_Push, Button_Switch_Keyboard:SW_Cherry_MX_1.00u_Plate, F.Cu at (-157.0, 302.3)
- added SW3: SW_Push, Button_Switch_Keyboard:SW_Cherry_MX_1.00u_Plate, F.Cu at (-141.9, 287.2)
- added SW4: SW_Push, Button_Switch_Keyboard:SW_Cherry_MX_1.00u_Plate, F.Cu at (-141.9, 302.3)
- added SW5: SW_Push, Button_Switch_Keyboard:SW_Cherry_MX_1.00u_Plate, F.Cu at (-126.8, 287.2)
- added SW6: SW_Push, Button_Switch_Keyboard:SW_Cherry_MX_1.00u_Plate, F.Cu at (-126.8, 302.3)
- added SW7: SW_Push, Button_Switch_Keyboard:SW_Cherry_MX_1.00u_Plate, F.Cu at (-111.8, 287.2)
- added SW8: SW_Push, Button_Switch_Keyboard:SW_Cherry_MX_1.00u_Plate, F.Cu at (-111.8, 302.3)
- added U1: Pico, MCU_RaspberryPi_and_Boards:RPi_Pico_SMD_TH, F.Cu at (-241.1, 214.5)
- added U2: 74HC4051, Package_DIP:SMDIP-16_W9.53mm, F.Cu at (-126.7, 143.5)
- added U3: PCF8574A, Package_DIP:SMDIP-16_W9.53mm, F.Cu at (-125.5, 264.6)
- added U4: PCF8574A, Package_DIP:SMDIP-16_W9.53mm, F.Cu at (-112.4, 264.6)
- added rotSW1: RotaryEncoder_Switch, Rotary_Encoder:RotaryEncoder_Alps_EC11E-Switch_Vertical_H20mm, F.Cu at (94.0, 124.5)
- added rotSW2: RotaryEncoder_Switch, Rotary_Encoder:RotaryEncoder_Alps_EC11E-Switch_Vertical_H20mm, F.Cu at (119.3, 124.5)
- added rotSW3: RotaryEncoder_Switch, Rotary_Encoder:RotaryEncoder_Alps_EC11E-Switch_Vertical_H20mm, F.Cu at (144.7, 124.5)
